File: Max100x100Plate.kicad_pcb (KiCad board)
At the start: 2 copper layers, 100 x 100 mm, 9 parts

Commit message: Add Defaults
Add predefined metric sizes for tracks and vias.  Theses are a good start for most small boards.
Other:
- rule pad_to_mask_clearance: 0.05 -> 0
Changed lines of the file:
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@@
       (dielectric_constraints no)
     )
-    (pad_to_mask_clearance 0.05)
-    (solder_mask_min_width 0.254)
+    (pad_to_mask_clearance 0)
     (pcbplotparams
       (layerselection 0x00010fc_ffffffff)
